File: PowerBoard/PowerBoard.kicad_sch (KiCad schematic)
At the start: 118 parts, among them J1 V_IN, J11 GND, J12 V_IN, J2 PH_B, J3 PH_A, J4 PH_C, J5 PH_B_CONNECTOR, J6 PH_A_CONNECTOR, J7 PH_C_CONNECTOR, Q1 HSP0076A, Q10 HSP0076A, Q11 HSP0076A, Q12 HSP0076A, Q13 HSP0076A, Q14 HSP0076A, Q15 HSP0076A, Q16 HSP0076A, Q17 HSP0076A, Q18 HSP0076A, Q2 HSP0076A, Q3 HSP0076A, Q4 HSP0076A, Q5 HSP0076A, Q6 HSP0076A, Q7 HSP0076A, Q8 HSP0076A, Q9 HSP0076A

Commit message: final
Parts:
- added C22, C23, C24: 470u_200V, Capacitor_THT:CP_Radial_D16.0mm_P7.50mm, symbol Device:C_Polarized_US
Connections:
- net GND: now also C22.2, C23.2, C24.2
- net V_IN: now also C22.1, C23.1, C24.1
- no-connect marks 6 -> 0
Changed lines of the file:
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@@
 		(color 0 0 0 0)
 	)
-	(no_connect
-		(at 186.69 153.67)
-	)
-	(no_connect
-		(at 186.69 146.05)
-	)
-	(no_connect
-		(at 201.93 146.05)
-	)
-	(no_connect
-		(at 256.54 153.67)
-	)
-	(no_connect
-		(at 201.93 153.67)
-	)
-	(no_connect
-		(at 256.54 146.05)
-	)
 	(wire
 		(pts
@@
 	)
 	(symbol
+		(lib_id "Device:C_Polarized_US")
+		(at 186.69 149.86 0)
+		(unit 1)
+		(exclude_from_sim no)
+		(in_bom yes)
+		(on_board yes)
+		(dnp no)
+		(property "Reference" "C24"
+			(at 187.96 147.32 0)
+			(effects
+				(font
+					(size 1.27 1.27)
+				)
+				(justify left)
+			)
+		)
+		(property "Value" "470u_200V"
+			(at 187.706 153.162 0)
+			(effects
+				(font
+					(size 1.27 1.27)
+				)
+				(justify left)
+			)
+		)
+		(property "Footprint" "Capacitor_THT:CP_Radial_D16.0mm_P7.50mm"
+			(at 186.69 149.86 0)
+			(effects
+				(font
+					(size 1.27 1.27)
+				)
+				(hide yes)
+			)
+		)
+		(property "Datasheet" "~"
+			(at 186.69 149.86 0)
+			(effects
+				(font
+					(size 1.27 1.27)
+				)
+				(hide yes)
+			)
+		)
+		(property "Description" "Polarized capacitor, US symbol"
+			(at 186.69 149.86 0)
+			(effects
+				(font
+					(size 1.27 1.27)
+				)
+				(hide yes)
+			)
+		)
+		(pin "2"
+		)
+		(pin "1"
+		)
+		(instances
+			(project "PowerBoard"
+				(path "/f0d46a6e-2214-493e-8380-6329d5bb9b12"
+					(reference "C24")
+					(unit 1)
+				)
+			)
+		)
+	)
+	(symbol
 		(lib_id "Diode:1N4148W")
 		(at 237.49 66.04 270)
@@
 	)
 	(symbol
+		(lib_id "Device:C_Polarized_US")
+		(at 201.93 149.86 0)
+		(unit 1)
+		(exclude_from_sim no)
+		(in_bom yes)
+		(on_board yes)
+		(dnp no)
+		(property "Reference" "C23"
+			(at 203.2 147.32 0)
+			(effects
+				(font
+					(size 1.27 1.27)
+				)
+				(justify left)
+			)
+		)
+		(property "Value" "470u_200V"
+			(at 202.946 153.162 0)
+			(effects
+				(font
+					(size 1.27 1.27)
+				)
+				(justify left)
+			)
+		)
+		(property "Footprint" "Capacitor_THT:CP_Radial_D16.0mm_P7.50mm"
+			(at 201.93 149.86 0)
+			(effects
+				(font
+					(size 1.27 1.27)
+				)
+				(hide yes)
+			)
+		)
+		(property "Datasheet" "~"
+			(at 201.93 149.86 0)
+			(effects
+				(font
+					(size 1.27 1.27)
+				)
+				(hide yes)
+			)
+		)
+		(property "Description" "Polarized capacitor, US symbol"
+			(at 201.93 149.86 0)
+			(effects
+				(font
+					(size 1.27 1.27)
+				)
+				(hide yes)
+			)
+		)
+		(pin "2"
+		)
+		(pin "1"
+		)
+		(instances
+			(project "PowerBoard"
+				(path "/f0d46a6e-2214-493e-8380-6329d5bb9b12"
+					(reference "C23")
+					(unit 1)
+				)
+			)
+		)
+	)
+	(symbol
 		(lib_id "power:PWR_FLAG")
 		(at 109.22 186.69 90)
@@
 					(unit 1)
 				)
+			)
+		)
+	)
+	(symbol
+		(lib_id "Device:C_Polarized_US")
+		(at 256.54 149.86 0)
+		(unit 1)
+		(exclude_from_sim no)
+		(in_bom yes)
+		(on_board yes)
+		(dnp no)
+		(property "Reference" "C22"
+			(at 257.81 147.32 0)
+			(effects
+				(font
+					(size 1.27 1.27)
+				)
+				(justify left)
+			)
+		)
+		(property "Value" "470u_200V"
+			(at 257.556 153.162 0)
+			(effects
+				(font
+					(size 1.27 1.27)
+				)
+				(justify left)
+			)
+		)
+		(property "Footprint" "Capacitor_THT:CP_Radial_D16.0mm_P7.50mm"
+			(at 256.54 149.86 0)
+			(effects
+				(font
+					(size 1.27 1.27)
+				)
+				(hide yes)
+			)
+		)
+		(property "Datasheet" "~"
+			(at 256.54 149.86 0)
+			(effects
+				(font
+					(size 1.27 1.27)
+				)
+				(hide yes)
+			)
+		)
+		(property "Description" "Polarized capacitor, US symbol"
+			(at 256.54 149.86 0)
+			(effects
+				(font
+					(size 1.27 1.27)
+				)
+				(hide yes)
+			)
+		)
+		(pin "2"
+		)
+		(pin "1"
+		)
+		(instances
+			(project "PowerBoard"
+				(path "/f0d46a6e-2214-493e-8380-6329d5bb9b12"
+					(reference "C22")
+					(unit 1)
+				)
